File: pcb/top-plate/top-plate.kicad_pcb (KiCad board)
At the start: 2 copper layers, 285.8 x 116.7 mm, 85 parts

Commit message: Update top plate footprints
Parts:
- added REF**: mx_top_plate_1.25u, bschwind_slots:mx_top_plate_1.25u, F.Cu at (231.0, 126.2)
- added REF**: mx_top_plate_1.25u, bschwind_slots:mx_top_plate_1.25u, F.Cu at (88.1, 126.2)

Commit message: Update the footprints for the top plate
Other:
- board text added: "JLCJLCJLCJLC"
- board text added: "key-ripper-top-plate v0.1"
