File: pcb/top-plate/top-plate.kicad_pcb (KiCad board)
At the start: 2 copper layers, 285.8 x 114.3 mm, 86 parts

Commit message: Change top plate cutouts to pcb-mounted stabilizer style
Parts:
- REF** (x2): footprint bschwind_slots:mx_top_plate_2.25u -> bschwind_slots:mx_top_plate_2.25u_pcb_mount
- REF**: footprint bschwind_slots:mx_top_plate_6.25u -> bschwind_slots:mx_top_plate_6.25u_pcb_mount
- REF**: footprint bschwind_slots:mx_top_plate_2.00u -> bschwind_slots:mx_top_plate_2.00u_pcb_mount
