File: pcb/key-ripper.kicad_sch (KiCad schematic)
At the start: 219 parts, among them J1 Conn_01x03, SW1 ESC, SW10 F9, SW11 F10, SW12 F11, SW13 F12, SW14 TILDE, SW15 1, SW16 2, SW17 3, SW18 4, SW19 5, SW2 F1, SW20 6, SW21 7, SW22 8, SW23 9, SW24 0, SW25 -, SW26 =, SW27 BACKSPACE, SW28 TAB, SW29 Q, SW3 F2, SW30 W, SW31 E, SW32 R, SW33 T, SW34 Y, SW35 U, SW36 I, SW37 O, SW38 P, SW39 [, SW4 F3, SW40 ], SW41 \, SW42 CAPS, SW43 A, SW44 S, SW45 D, SW46 F, SW47 G, SW48 H, SW49 J, SW5 F4, SW50 K, SW51 L, SW52 ;, SW53 ', SW54 ENTER, SW55 L_SHIFT, SW56 Z, SW57 X, SW58 C, SW59 V, SW6 F5, SW60 B, SW61 N, SW62 M, SW63 ,, SW64 ., SW65 /, SW66 UP, SW67 FN, SW68 BL_CTRL, SW69 L_ALT, SW7 F6, SW70 L_CMD, SW71 SPACE, SW72 R_CMD, SW73 LEFT, SW74 DOWN, SW75 RIGHT, SW8 F7, SW9 F8, U1 RP2040, U2 TYPE-C-31-M-12, U3 XC6206PxxxMR, U4 W25Q128JVS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

Commit message: Change the crystal capacitor footprints to 1608 metric size
Parts:
- C6, C7: footprint Capacitor_SMD:C_0402_1005Metric -> Capacitor_SMD:C_0603_1608Metric
Changed lines of the file:
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@@
       (effects (font (size 1.27 1.27)) (justify left))
     )
-    (property "Footprint" "Capacitor_SMD:C_0402_1005Metric" (id 2) (at 147.32 125.73 0)
+    (property "Footprint" "Capacitor_SMD:C_0603_1608Metric" (id 2) (at 147.32 125.73 0)
       (effects (font (size 1.27 1.27)) hide)
     )
@@
       (effects (font (size 1.27 1.27)) (justify left))
     )
-    (property "Footprint" "Capacitor_SMD:C_0402_1005Metric" (id 2) (at 135.255 125.73 0)
+    (property "Footprint" "Capacitor_SMD:C_0603_1608Metric" (id 2) (at 135.255 125.73 0)
       (effects (font (size 1.27 1.27)) hide)
     )
@@
     )
     (path "/d71055b4-8d7d-4df8-9391-f9729ebb8303"
-      (reference "C6") (unit 1) (value "30pF") (footprint "Capacitor_SMD:C_0402_1005Metric")
+      (reference "C6") (unit 1) (value "30pF") (footprint "Capacitor_SMD:C_0603_1608Metric")
     )
     (path "/5aa29279-90fb-4e4c-904d-0a1a183027af"
-      (reference "C7") (unit 1) (value "30pF") (footprint "Capacitor_SMD:C_0402_1005Metric")
+      (reference "C7") (unit 1) (value "30pF") (footprint "Capacitor_SMD:C_0603_1608Metric")
     )
     (path "/f114f220-3a87-49ce-835f-d98a152486aa"
